File: stepper_controller_5x3.kicad_pcb (KiCad board)
At the start: 2 copper layers, 121.3 x 67.3 mm, 76 parts, among them P1 PWR_JACK_2.5x5.5, T1 TERM_BLK_HDR_4POS_VERT_0.2IN, T2 TERM_BLK_HDR_4POS_VERT_0.150IN, T3 TERM_BLK_HDR_4POS_VERT_0.2IN, T4 TERM_BLK_HDR_4POS_VERT_0.150IN, T5 TERM_BLK_HDR_4POS_VERT_0.2IN, T6 TERM_BLK_HDR_4POS_VERT_0.150IN, U1 TMC429, U2 SN74ABT541BDWR, U3 MAX6817, U4 MAX6817, U5 MAX6817

Commit message: Test routing of new version
Parts:
- removed C18, C22, C23, C24, C25: 470pF, stepper_controller_5x3:SM0805
- removed C19, C26: 0.1uF, stepper_controller_5x3:SM1210
- removed C20: 220uF_POL, stepper_controller_5x3:C_ELEC_10
- removed C21: 10uF, stepper_controller_5x3:SM1210
- removed L1, L10, L11, L12, L2, L3, L4, L5, L6, L7, L8, L9: 90nH, stepper_controller_5x3:ECS-MPI4040
- removed RV1, RV10, RV11, RV12, RV13, RV14, RV15, RV16, RV17, RV18, RV2, RV3, RV4, RV5, RV6, RV7, RV8, RV9: VAR, stepper_controller_5x3:SM0805
- added R10: 845, stepper_controller_5x3:SM0805, B.Cu at (137.8, 131.4)
- added R11: 845, stepper_controller_5x3:SM0805, B.Cu at (137.8, 120.0)
- added R12: 10.0k, footprints:SM0805, B.Cu at (99.1, 95.9)
- added R13: 845, stepper_controller_5x3:SM0805, B.Cu at (104.8, 127.6)
- added R14: 845, stepper_controller_5x3:SM0805, B.Cu at (97.2, 120.0)
- added R15: 845, stepper_controller_5x3:SM0805, B.Cu at (104.8, 131.4)
- added R16: 845, stepper_controller_5x3:SM0805, B.Cu at (104.8, 120.0)
- added R2: 10.0k, footprints:SM0805, B.Cu at (165.1, 95.9)
- added R3: 845, stepper_controller_5x3:SM0805, B.Cu at (170.8, 127.6)
- added R4: 845, stepper_controller_5x3:SM0805, B.Cu at (163.2, 120.0)
- added R5: 845, stepper_controller_5x3:SM0805, B.Cu at (170.8, 131.4)
- added R6: 845, stepper_controller_5x3:SM0805, B.Cu at (170.8, 120.0)
- added R7: 10.0k, footprints:SM0805, B.Cu at (132.1, 95.9)
- added R8: 845, stepper_controller_5x3:SM0805, B.Cu at (137.8, 127.6)
- added R9: 845, stepper_controller_5x3:SM0805, B.Cu at (130.2, 120.0)
- added U10: BUFFER_TRI_STATE, stepper_controller_5x3:SOT-23-5, B.Cu at (99.1, 99.7)
- added U11: OPTOISO_2CHAN, stepper_controller_5x3:SO-8, B.Cu at (99.1, 129.5)
- added U12: MAX6817, stepper_controller_5x3:MAX6817, B.Cu at (87.0, 129.5)
- added U6: MAX6817, stepper_controller_5x3:MAX6817, B.Cu at (153.0, 129.5)
- added U7: BUFFER_TRI_STATE, stepper_controller_5x3:SOT-23-5, B.Cu at (132.1, 99.7)
- added U8: OPTOISO_2CHAN, stepper_controller_5x3:SO-8, B.Cu at (132.1, 129.5)
- added U9: MAX6817, stepper_controller_5x3:MAX6817, B.Cu at (120.0, 129.5)
- C10: value 470pF -> 220uF_POL; footprint stepper_controller_5x3:SM0805 -> stepper_controller_5x3:C_ELEC_10; moved to F.Cu
- C11, C15: value 470pF -> 10uF; footprint stepper_controller_5x3:SM0805 -> stepper_controller_5x3:SM1210
- C13: value 220uF_POL -> 0.1uF; footprint stepper_controller_5x3:C_ELEC_10 -> stepper_controller_5x3:SM1210; moved to B.Cu
- C14: value 10uF -> 220uF_POL; footprint stepper_controller_5x3:SM1210 -> stepper_controller_5x3:C_ELEC_10; moved to F.Cu
- C16, C17, C8, C9: value 470pF -> 0.1uF; footprint stepper_controller_5x3:SM0805 -> stepper_controller_5x3:SM1210
- R1: value 1k -> 10.0k; footprint stepper_controller_5x3:SM1210 -> footprints:SM0805
- U2: value SN74ABT541BDWR -> BUFFER_TRI_STATE; footprint stepper_controller_5x3:SOIC_20 -> stepper_controller_5x3:SOT-23-5
- U3: value MAX6817 -> SN74ABT541BDWR; footprint stepper_controller_5x3:MAX6817 -> stepper_controller_5x3:SOIC_20
- U4: value MAX6817 -> BUFFER_TRI_STATE; footprint stepper_controller_5x3:MAX6817 -> stepper_controller_5x3:SOT-23-5
- U5: value MAX6817 -> OPTOISO_2CHAN; footprint stepper_controller_5x3:MAX6817 -> stepper_controller_5x3:SO-8
- moved U3 77.5 mm to (88.9, 114.3), turned to 90 degrees
- moved C17 68.3 mm to (81.9, 129.5), turned to 270 degrees
- moved C16 66.6 mm to (92.1, 129.5), turned to 270 degrees
- moved U5 66.1 mm to (165.1, 129.5)
- moved C9 54.4 mm to (148.0, 129.5), turned to 270 degrees
- moved C8 51.9 mm to (158.1, 129.5), turned to 270 degrees
- moved C15 50.5 mm to (91.4, 97.8), turned to 0 degrees
- moved C10 49.8 mm to (115.6, 99.1)
- moved C12 45.7 mm to (125.1, 129.5), turned to 270 degrees
- moved U4 43.7 mm to (165.1, 99.7), turned to 180 degrees
- moved C14 42.0 mm to (82.5, 99.1), turned to 90 degrees
- moved C11 38.9 mm to (124.5, 97.8), turned to 0 degrees
- moved R1 34.8 mm to (111.8, 122.6), turned to 90 degrees
- moved C13 30.5 mm to (114.9, 129.5), turned to 270 degrees
- moved U2 27.3 mm to (115.6, 122.6), turned to 270 degrees
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Connections:
- C10 pad 1: /tmc429_driver_0/stepper_0/B_+F -> VAA
- C11 pad 1: /tmc429_driver_0/stepper_0/B_-F -> VAA
- C13 pad 1: VAA -> +3V3
- C15 pad 1: /tmc429_driver_0/stepper_1/A_+F -> VAA
- C16 pad 1: /tmc429_driver_0/stepper_1/A_-F -> +3V3
- C17 pad 1: /tmc429_driver_0/stepper_1/B_+F -> +3V3
- C8 pad 1: /tmc429_driver_0/stepper_0/A_+F -> +3V3
- C9 pad 1: /tmc429_driver_0/stepper_0/A_-F -> +3V3
- MDB1 pad 23: +5V -> (no net)
- R1 pad 1: +5V -> +3V3
- R1 pad 2: GND -> /CS_429
- SS1 pad 4: /MISO -> /tmc429_driver_0/stepper_0/MISO_UB
- SS2 pad 4: /MISO -> /tmc429_driver_0/stepper_1/MISO_UB
- SS3 pad 4: /MISO -> /tmc429_driver_0/stepper_2/MISO_UB
- T1 pad 1: /tmc429_driver_0/stepper_0/B_-F -> /tmc429_driver_0/stepper_0/B_-
- T1 pad 2: /tmc429_driver_0/stepper_0/B_+F -> /tmc429_driver_0/stepper_0/B_+
- T1 pad 3: /tmc429_driver_0/stepper_0/A_-F -> /tmc429_driver_0/stepper_0/A_-
- T1 pad 4: /tmc429_driver_0/stepper_0/A_+F -> /tmc429_driver_0/stepper_0/A_+
- T2 pad 2: GND -> /tmc429_driver_0/stepper_0/REF_GND
- T2 pad 4: GND -> /tmc429_driver_0/stepper_0/REFR_GND
- T3 pad 1: /tmc429_driver_0/stepper_1/B_-F -> /tmc429_driver_0/stepper_1/B_-
- T3 pad 2: /tmc429_driver_0/stepper_1/B_+F -> /tmc429_driver_0/stepper_1/B_+
- T3 pad 3: /tmc429_driver_0/stepper_1/A_-F -> /tmc429_driver_0/stepper_1/A_-
- T3 pad 4: /tmc429_driver_0/stepper_1/A_+F -> /tmc429_driver_0/stepper_1/A_+
- T4 pad 2: GND -> /tmc429_driver_0/stepper_1/REF_GND
- T4 pad 4: GND -> /tmc429_driver_0/stepper_1/REFR_GND
- T5 pad 1: /tmc429_driver_0/stepper_2/B_-F -> /tmc429_driver_0/stepper_2/B_-
- T5 pad 2: /tmc429_driver_0/stepper_2/B_+F -> /tmc429_driver_0/stepper_2/B_+
- T5 pad 3: /tmc429_driver_0/stepper_2/A_-F -> /tmc429_driver_0/stepper_2/A_-
- T5 pad 4: /tmc429_driver_0/stepper_2/A_+F -> /tmc429_driver_0/stepper_2/A_+
- T6 pad 2: GND -> /tmc429_driver_0/stepper_2/REF_GND
- T6 pad 4: GND -> /tmc429_driver_0/stepper_2/REFR_GND
- U1 pad 12: /MISO -> /tmc429_driver_0/MISO_UB
- U2 pad 1: GND -> /CS_429
- U2 pad 2: /SCK -> /tmc429_driver_0/MISO_UB
- U2 pad 3: /MOSI -> GND
- U2 pad 4: /ENABLE_0 -> /MISO
- U2 pad 5: /CS_DRIVER_0 -> +3V3
- U3 pad 1: /tmc429_driver_0/stepper_0/REF_B -> GND
- U3 pad 2: GND -> /SCK
- U3 pad 3: /tmc429_driver_0/stepper_0/REFR_B -> /MOSI
- U3 pad 4: /tmc429_driver_0/REFR_0 -> /ENABLE_0
- U3 pad 5: +3V3 -> /CS_DRIVER_0
- U3 pad 6: /tmc429_driver_0/REF_0 -> /ENABLE_1
- U4 pad 1: /tmc429_driver_0/stepper_1/REF_B -> /tmc429_driver_0/~CS_DRIVER_0_B
- U4 pad 2: GND -> /tmc429_driver_0/stepper_0/MISO_UB
- U4 pad 3: /tmc429_driver_0/stepper_1/REFR_B -> GND
- U4 pad 4: /tmc429_driver_0/REFR_1 -> /MISO
- U5 pad 1: /tmc429_driver_0/stepper_2/REF_B -> /tmc429_driver_0/stepper_0/REF_PWR
- U5 pad 2: GND -> /tmc429_driver_0/stepper_0/REF_B
- U5 pad 3: /tmc429_driver_0/stepper_2/REFR_B -> /tmc429_driver_0/stepper_0/REFR_B
- U5 pad 4: /tmc429_driver_0/REFR_2 -> /tmc429_driver_0/stepper_0/REFR_PWR
- U5 pad 5: +3V3 -> GND
- U5 pad 6: /tmc429_driver_0/REF_2 -> /tmc429_driver_0/stepper_0/REFR_BI
Routing:
- net GND: track 0.00 -> 510.9 mm, vias 0 -> 3
- net +3V3: track 0.00 -> 299.6 mm, vias 0 -> 6
- net +5V: track 0.00 -> 254.2 mm, vias 0 -> 1
- net /MISO: track 0.00 -> 186.6 mm, vias 0 -> 3
- net VAA: track 0.00 -> 175.7 mm
- net /tmc429_driver_0/~CS_DRIVER_0_B: track 0.00 -> 96.8 mm, vias 0 -> 1
- net /tmc429_driver_0/MOSI_B: track 0.00 -> 81.7 mm
- net /tmc429_driver_0/SCK_B: track 0.00 -> 81.0 mm
- net /INT: track 0.00 -> 79.2 mm
- net /tmc429_driver_0/~ENABLE_0_B: track 0.00 -> 77.2 mm, vias 0 -> 1
- net /MOSI: track 0.00 -> 76.7 mm, vias 0 -> 2
- net /ENABLE_2: track 0.00 -> 70.4 mm
- net /tmc429_driver_0/STEP_0: track 0.00 -> 68.8 mm, vias 0 -> 1
- net /tmc429_driver_0/DIR_0: track 0.00 -> 68.3 mm, vias 0 -> 1
- net /ENABLE_1: track 0.00 -> 63.5 mm
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- added copper zone on B.Cu, net GND
- added copper zone on F.Cu, net VAA
Other:
- board text added: "Janelia Modular Device stepper_controller part_number: 1140 04/2019 ver 1.2 5x3"
- board text removed: "Janelia Modular Device stepper_controller part_number: 1140 03/2019 ver 1.2 5x3"
